Commit message: Gripper

File: URDF/DexArm.urdf (robot description, URDF)
Before this commit: robot DexArm_unofficial, 9 links, 8 joints
Links:
- removed link Suction
- added link GripperAxis; collision mesh filename=./STL/M02-GripperAxis.stl scale=0.001 0.001 0.001; visual mesh filename=./STL/M02-GripperAxis.stl scale=0.001 0.001 0.001
- added link GripperFingerA1; collision mesh filename=./STL/M02-GripperFinger1.stl scale=0.001 0.001 0.001; visual mesh filename=./STL/M02-GripperFinger1.stl scale=0.001 0.001 0.001
- added link GripperFingerA2; collision mesh filename=./STL/M02-GripperFinger2.stl scale=0.001 0.001 0.001; visual mesh filename=./STL/M02-GripperFinger2.stl scale=0.001 0.001 0.001
- added link GripperFingerA3; collision mesh filename=./STL/M02-GripperFinger3.stl scale=0.001 0.001 0.001; visual mesh filename=./STL/M02-GripperFinger3.stl scale=0.001 0.001 0.001
- added link GripperFingerA4; collision mesh filename=./STL/M02-GripperFinger4.stl scale=0.001 0.001 0.001; visual mesh filename=./STL/M02-GripperFinger4.stl scale=0.001 0.001 0.001
- added link GripperFingerA5; collision mesh filename=./STL/M02-GripperFinger5.stl scale=0.001 0.001 0.001; visual mesh filename=./STL/M02-GripperFinger5.stl scale=0.001 0.001 0.001
- added link GripperFingerB1; collision mesh filename=./STL/M02-GripperFinger1.stl scale=0.001 0.001 0.001; visual mesh filename=./STL/M02-GripperFinger1.stl scale=0.001 0.001 0.001
- added link GripperFingerB2; collision mesh filename=./STL/M02-GripperFinger2.stl scale=0.001 0.001 0.001; visual mesh filename=./STL/M02-GripperFinger2.stl scale=0.001 0.001 0.001
- added link GripperFingerB3; collision mesh filename=./STL/M02-GripperFinger3.stl scale=0.001 0.001 0.001; visual mesh filename=./STL/M02-GripperFinger3.stl scale=0.001 0.001 0.001
- added link GripperFingerB4; collision mesh filename=./STL/M02-GripperFinger4.stl scale=0.001 0.001 0.001; visual mesh filename=./STL/M02-GripperFinger4.stl scale=0.001 0.001 0.001
- added link GripperFingerB5; collision mesh filename=./STL/M02-GripperFinger5.stl scale=0.001 0.001 0.001; visual mesh filename=./STL/M02-GripperFinger5.stl scale=0.001 0.001 0.001
- added link GripperFingerC1; collision mesh filename=./STL/M02-GripperFinger1.stl scale=0.001 0.001 0.001; visual mesh filename=./STL/M02-GripperFinger1.stl scale=0.001 0.001 0.001
- added link GripperFingerC2; collision mesh filename=./STL/M02-GripperFinger2.stl scale=0.001 0.001 0.001; visual mesh filename=./STL/M02-GripperFinger2.stl scale=0.001 0.001 0.001
- added link GripperFingerC3; collision mesh filename=./STL/M02-GripperFinger3.stl scale=0.001 0.001 0.001; visual mesh filename=./STL/M02-GripperFinger3.stl scale=0.001 0.001 0.001
- added link GripperFingerC4; collision mesh filename=./STL/M02-GripperFinger4.stl scale=0.001 0.001 0.001; visual mesh filename=./STL/M02-GripperFinger4.stl scale=0.001 0.001 0.001
- added link GripperFingerC5; collision mesh filename=./STL/M02-GripperFinger5.stl scale=0.001 0.001 0.001; visual mesh filename=./STL/M02-GripperFinger5.stl scale=0.001 0.001 0.001
- added link GripperMount; collision mesh filename=./STL/M02-GripperMount.stl scale=0.001 0.001 0.001; visual mesh filename=./STL/M02-GripperMount.stl scale=0.001 0.001 0.001
Joints:
- removed joint EE->Suction
- added joint EE->GripperMount: type fixed, parent EE, child GripperMount, origin xyz=0 -0.05 0.01 rpy=0 0 0, axis 1 0 0, limit lower=-0.6 upper=1.2 effort=30 velocity=1.74533
- added joint GripperAxis->GripperFingerA1: type fixed, parent GripperAxis, child GripperFingerA1, origin xyz=-0.020 0.00 -0.042 rpy=0 0 0, axis 0 0 1, limit effort=30 velocity=1.74533
- added joint GripperAxis->GripperFingerB1: type fixed, parent GripperAxis, child GripperFingerB1, origin xyz=0.010 0.018 -0.042 rpy=0 0 0.0, axis 0 0 1, limit effort=30 velocity=1.74533
- added joint GripperAxis->GripperFingerC1: type fixed, parent GripperAxis, child GripperFingerC1, origin xyz=0.010 -0.017 -0.042 rpy=0 0 0, axis 0 0 1, limit effort=30 velocity=1.74533
- added joint GripperFingerA1->GripperFingerA2: type revolute, parent GripperFingerA1, child GripperFingerA2, origin xyz=0.003 0.00 -0.008 rpy=0 0 0, axis 0 1 0, limit lower=-0.3 upper=0.0 effort=30 velocity=1.74533
- added joint GripperFingerA2->GripperFingerA3: type revolute, parent GripperFingerA2, child GripperFingerA3, origin xyz=0.0005 0.00 -0.007 rpy=0 0 0, axis 0 1 0, limit lower=-0.3 upper=0.0 effort=30 velocity=1.74533, mimic joint=GripperFingerA1->GripperFingerA2 multiplier=1 offset=0
- added joint GripperFingerA3->GripperFingerA4: type revolute, parent GripperFingerA3, child GripperFingerA4, origin xyz=0.0005 0.00 -0.007 rpy=0 0 0, axis 0 1 0, limit lower=-0.3 upper=0.0 effort=30 velocity=1.74533, mimic joint=GripperFingerA1->GripperFingerA2 multiplier=1 offset=0
- added joint GripperFingerA4->GripperFingerA5: type revolute, parent GripperFingerA4, child GripperFingerA5, origin xyz=0.0005 0.00 -0.007 rpy=0 0 0, axis 0 1 0, limit lower=-0.3 upper=0.0 effort=30 velocity=1.74533, mimic joint=GripperFingerA1->GripperFingerA2 multiplier=1 offset=0
- added joint GripperFingerB1->GripperFingerB2: type revolute, parent GripperFingerB1, child GripperFingerB2, origin xyz=-0.003 -0.003 -0.008 rpy=0 0 1.1, axis 0 1 0, limit lower=0.0 upper=0.3 effort=30 velocity=1.74533, mimic joint=GripperFingerA1->GripperFingerA2 multiplier=-1 offset=0
- added joint GripperFingerB2->GripperFingerB3: type revolute, parent GripperFingerB2, child GripperFingerB3, origin xyz=-0.000 -0.000 -0.006 rpy=0 0 0.0, axis 0 1 0, limit lower=0 upper=0.3 effort=30 velocity=1.74533, mimic joint=GripperFingerA1->GripperFingerA2 multiplier=-1 offset=0
- added joint GripperFingerB3->GripperFingerB4: type revolute, parent GripperFingerB3, child GripperFingerB4, origin xyz=0.0005 0.00 -0.007 rpy=0 0 0.0, axis 0 1 0, limit lower=0. upper=0.3 effort=30 velocity=1.74533, mimic joint=GripperFingerA1->GripperFingerA2 multiplier=-1 offset=0
- added joint GripperFingerB4->GripperFingerB5: type revolute, parent GripperFingerB4, child GripperFingerB5, origin xyz=0.0005 0.00 -0.007 rpy=0 0 0, axis 0 1 0, limit lower=0 upper=0.3 effort=30 velocity=1.74533, mimic joint=GripperFingerA1->GripperFingerA2 multiplier=-1 offset=0
- added joint GripperFingerC1->GripperFingerC2: type revolute, parent GripperFingerC1, child GripperFingerC2, origin xyz=0.00 0.00 -0.008 rpy=0 0 2.1, axis 0 1 0, limit lower=-0.3 upper=0 effort=30 velocity=1.74533, mimic joint=GripperFingerA1->GripperFingerA2 multiplier=1 offset=0
- added joint GripperFingerC2->GripperFingerC3: type revolute, parent GripperFingerC2, child GripperFingerC3, origin xyz=0.0005 0.00 -0.006 rpy=0 0 0, axis 0 1 0, limit lower=-0.3 upper=0.0 effort=30 velocity=1.74533, mimic joint=GripperFingerA1->GripperFingerA2 multiplier=1 offset=0
- added joint GripperFingerC3->GripperFingerC4: type revolute, parent GripperFingerC3, child GripperFingerC4, origin xyz=0.0005 0.00 -0.007 rpy=0 0 0, axis 0 1 0, limit lower=-0.3 upper=0.0 effort=30 velocity=1.74533, mimic joint=GripperFingerA1->GripperFingerA2 multiplier=1 offset=0
- added joint GripperFingerC4->GripperFingerC5: type revolute, parent GripperFingerC4, child GripperFingerC5, origin xyz=0.0005 0.00 -0.007 rpy=0 0 0, axis 0 1 0, limit lower=-0.3 upper=0.0 effort=30 velocity=1.74533, mimic joint=GripperFingerA1->GripperFingerA2 multiplier=1 offset=0
- added joint GripperMount->GripperAxis: type continuous, parent GripperMount, child GripperAxis, origin xyz=-0.002 -0.06 0.0 rpy=0 0 0, axis 0 0 1, limit effort=30 velocity=1.74533
